Commit message: with gripper v1.0

File: install/gz_ros2_control_demos/share/gz_ros2_control_demos/urdf/test_gripper_mimic_joint_effort.xacro.urdf (robot description, URDF)
Before this commit: robot gripper, 4 links, 3 joints
Links:
- removed link base
- removed link world
- added link gripper_base, mass 0.5; collision box size=0.05 0.1 0.1; visual box size=0.05 0.1 0.1
- link finger_left: mass 4 -> 0.04; geometry collision box size=0.04 0.01 0.1; visual box size=0.04 0.01 0.1
- link finger_right: mass 4 -> 0.04; geometry collision box size=0.04 0.01 0.1; visual box size=0.04 0.01 0.1
Joints:
- removed joint world_to_base
- joint left_finger_joint: limit lower=0 upper=0.38 effort=1000.0 velocity=10 -> lower=0 upper=0.02 effort=10.0 velocity=0.1; origin xyz=0.0 0.48 1 rpy=0.0 0.0 3.1415926535 -> xyz=0 0.055 0.1 rpy=0.0 0.0 3.1415926535; parent base -> gripper_base
- joint right_finger_joint: limit lower=0 upper=0.38 effort=1000.0 velocity=10 -> lower=0 upper=0.02 effort=10.0 velocity=0.1; origin xyz=0.0 -0.48 1 rpy=0.0 0.0 0.0 -> xyz=0 -0.055 0.1 rpy=0.0 0.0 0.0; parent base -> gripper_base

File: install/gz_ros2_control_demos/share/gz_ros2_control_demos/urdf/test_gripper_mimic_joint_position.xacro.urdf (robot description, URDF)
Before this commit: robot gripper, 4 links, 3 joints
Links:
- removed link base
- removed link world
- added link gripper_base, mass 0.5; collision box size=0.05 0.1 0.1; visual box size=0.05 0.1 0.1
- link finger_left: mass 4 -> 0.04; geometry visual box size=0.04 0.01 0.1
- link finger_right: mass 4 -> 0.04; geometry visual box size=0.04 0.01 0.1
Joints:
- removed joint world_to_base
- joint left_finger_joint: axis 0 1 0 -> (none); limit lower=0 upper=0.38 effort=1000.0 velocity=10 -> (none); mimic joint=right_finger_joint -> (none); origin xyz=0.0 0.48 1 rpy=0.0 0.0 3.1415926535 -> xyz=0.0 0.048 0.1 rpy=0.0 0.0 3.1415926535; parent base -> gripper_base; type prismatic -> fixed
- joint right_finger_joint: limit lower=0 upper=0.38 effort=1000.0 velocity=10 -> lower=0 upper=0.086 effort=10.0 velocity=0.1; origin xyz=0.0 -0.48 1 rpy=0.0 0.0 0.0 -> xyz=0.0 -0.048 0.1 rpy=0.0 0.0 0.0; parent base -> gripper_base

File: install/ur_moveit_config/share/ur_moveit_config/srdf/ur_macro.srdf.xacro (robot description, xacro)
@@ -14,4 +14,9 @@
       <chain base_link="base_link" tip_link="tool0" />
     </group>
+    <group name="gripper">
+      <joint name="right_finger_joint"/>  # Primary joint
+      <joint name="left_finger_joint"/>   # Mimic joint
+    </group>
+    <end_effector name="gripper_ee" parent_link="gripper_base" group="gripper"/>
     <!--GROUP STATES - Purpose - Define a named state for a particular group, in terms of joint values. This is useful to define states like 'folded arms'-->
     <group_state name="home" group="ur_manipulator">
@@ -39,5 +44,10 @@
       <joint name="wrist_3_joint" value="-0.11" />
     </group_state>
-    <!--END EFFECTOR - Purpose - Represent information about an end effector.-->
+    <group_state name="open" group="gripper">
+      <joint name="right_finger_joint" value="0.004" />
+    </group_state>
+    <group_state name="close" group="gripper">
+      <joint name="right_finger_joint" value="0.085" />
+    </group_state>
     <!--VIRTUAL JOINT - Purpose - this element defines a virtual joint between a robot link and an external frame of reference (considered fixed with respect to the robot)-->
     <!--DISABLE COLLISIONS - By default it is assumed that any link of the robot could potentially come into collision with any other link in the robot. This tag disables collision checking between a specified pair of links. -->

File: install/ur_simulation_gz/share/ur_simulation_gz/urdf/ur_gz.ros2_control.xacro (robot description, xacro)
@@ -1,4 +1,5 @@
 <?xml version="1.0"?>
 <robot xmlns:xacro="http://www.ros.org/wiki/xacro">
+  <!-- Include the standard UR arm joint control description -->
   <xacro:include filename="$(find ur_description)/urdf/inc/ur_joint_control.xacro" />
   <xacro:macro name="ur_ros2_control" params="
@@ -6,18 +7,38 @@
     tf_prefix
     transmission_hw_interface:=hardware_interface/PositionJointInterface
-    initial_positions:=${dict(shoulder_pan_joint=0.0,shoulder_lift_joint=-1.57,elbow_joint=0.0,wrist_1_joint=-1.57,wrist_2_joint=0.0,wrist_3_joint=0.0)}
-    ">
-    <!-- Add URDF transmission elements (for ros_control) -->
-    <!--<xacro:ur_arm_transmission prefix="${prefix}" hw_interface="${transmission_hw_interface}" />-->
-    <!-- Placeholder for ros2_control transmission which don't yet exist -->
+    initial_positions:=${dict(
+      shoulder_pan_joint=0.0,
+      shoulder_lift_joint=-1.57,
+      elbow_joint=0.0,
+      wrist_1_joint=-1.57,
+      wrist_2_joint=0.0,
+      wrist_3_joint=0.0
+    )}
+  ">
+    <!-- Single hardware plugin for everything -->
     <ros2_control name="${name}" type="system">
       <hardware>
         <plugin>gz_ros2_control/GazeboSimSystem</plugin>
       </hardware>
+      <!-- UR Arm Joints -->
       <xacro:ur_joint_control_description
         tf_prefix="${tf_prefix}"
         initial_positions="${initial_positions}"
       />
-      </ros2_control>
+      <!-- Gripper Finger Joints -->
+      <joint name="right_finger_joint">
+        <command_interface name="position"/>
+        <param name="p">100.0</param>
+        <param name="i">1.0</param>
+        <param name="d">10.0</param>
+        <state_interface name="position">
+          <param name="initial_value">0.004</param>
+        </state_interface>
+        <state_interface name="velocity"/>
+        <state_interface name="effort"/>
+        <state_interface name="acceleration"/>
+        <state_interface name="deceleration"/>
+      </joint>
+    </ros2_control>
   </xacro:macro>
 </robot>

File: install/ur_simulation_gz/share/ur_simulation_gz/urdf/ur_gz.urdf.xacro (robot description, xacro)
@@ -6,4 +6,5 @@
   <xacro:include filename="$(find ur_description)/urdf/ur_macro.xacro"/>
   <xacro:include filename="$(find ur_simulation_gz)/urdf/ur_gz.ros2_control.xacro" />
+  <xacro:include filename="$(find gz_ros2_control_demos)/urdf/test_gripper_mimic_joint_position.xacro.urdf" />
   <!-- possible 'ur_type' values: ur3, ur3e, ur5, ur5e, ur10, ur10e, ur16e, ur20, ur30 -->
   <!-- the default value should raise an error in case this was called without defining the type -->
@@ -60,6 +61,10 @@
     <origin xyz="1.06135 0.73380 1.100" rpy="0 0 3.1416" />          <!-- position robot in the world -->
   </xacro:ur_robot>
-  <gazebo reference="world">
-  </gazebo>
+  <joint name="tool0_to_gripper_base" type="fixed">
+    <parent link="tool0"/>  <!-- UR5's end-effector -->
+    <child link="gripper_base"/>    <!-- Gripper's base link -->
+    <origin xyz="0 0 0.0001" rpy="0 0 0"/> <!-- Adjust offset if needed -->
+  </joint>
+  <gazebo reference="world"></gazebo>
   <gazebo>
     <plugin filename="gz_ros2_control-system" name="gz_ros2_control::GazeboSimROS2ControlPlugin">
